File: Echo Cinematic/AUDIO IN.kicad_sch (KiCad schematic)
At the start: 17 parts, among them J16 Input R, J8 Input L, U2 TL072

Commit message: Added input jack switching circuits, fab files updated and finalized.
Parts:
- added R51, R52: 0R, Resistor_SMD:R_0603_1608Metric, symbol Device:R_Small
Connections:
- net AUDIO_IN_L: now also R51.1
- net AUDIO_IN_R: now also R52.2
- net at J8.TN: now also R52.1
- net at J16.TN: now also R51.2
- no-connect marks 2 -> 0
Changed lines of the file:
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@@
 (kicad_sch (version 20230121) (generator eeschema)
   (paper "A4")
+  (junction (at 53.34 107.95) (diameter 0) (color 0 0 0 0)
+  )
   (junction (at 96.52 107.95) (diameter 0) (color 0 0 0 0)
   )
@@
   (junction (at 243.84 130.81) (diameter 0) (color 0 0 0 0)
   )
+  (junction (at 48.26 53.34) (diameter 0) (color 0 0 0 0)
+  )
   (junction (at 118.11 44.45) (diameter 0) (color 0 0 0 0)
   )
@@
   (junction (at 118.11 110.49) (diameter 0) (color 0 0 0 0)
   )
-  (no_connect (at 41.91 110.49))
-  (no_connect (at 41.91 55.88))
   (wire (pts (xy 44.45 62.23) (xy 36.83 62.23))
     (stroke (width 0) (type default))
@@
     (stroke (width 0) (type default))
   )
+  (wire (pts (xy 53.34 78.74) (xy 53.34 55.88))
+    (stroke (width 0) (type default))
+  )
   (wire (pts (xy 118.11 35.56) (xy 118.11 44.45))
     (stroke (width 0) (type default))
@@
     (stroke (width 0) (type default))
   )
+  (wire (pts (xy 48.26 110.49) (xy 41.91 110.49))
+    (stroke (width 0) (type default))
+  )
   (wire (pts (xy 90.17 107.95) (xy 96.52 107.95))
     (stroke (width 0) (type default))
@@
     (stroke (width 0) (type default))
   )
+  (wire (pts (xy 53.34 107.95) (xy 71.12 107.95))
+    (stroke (width 0) (type default))
+  )
   (wire (pts (xy 118.11 99.06) (xy 118.11 110.49))
     (stroke (width 0) (type default))
@@
     (stroke (width 0) (type default))
   )
-  (wire (pts (xy 41.91 107.95) (xy 71.12 107.95))
+  (wire (pts (xy 41.91 107.95) (xy 53.34 107.95))
     (stroke (width 0) (type default))
   )
@@
     (stroke (width 0) (type default))
   )
-  (wire (pts (xy 41.91 53.34) (xy 71.12 53.34))
+  (wire (pts (xy 41.91 53.34) (xy 48.26 53.34))
     (stroke (width 0) (type default))
   )
@@
     (stroke (width 0) (type default))
   )
+  (wire (pts (xy 53.34 55.88) (xy 41.91 55.88))
+    (stroke (width 0) (type default))
+  )
   (wire (pts (xy 96.52 44.45) (xy 96.52 53.34))
     (stroke (width 0) (type default))
@@
     (stroke (width 0) (type default))
   )
+  (wire (pts (xy 48.26 53.34) (xy 71.12 53.34))
+    (stroke (width 0) (type default))
+  )
+  (wire (pts (xy 53.34 83.82) (xy 53.34 107.95))
+    (stroke (width 0) (type default))
+  )
   (wire (pts (xy 96.52 53.34) (xy 100.33 53.34))
     (stroke (width 0) (type default))
@@
     (stroke (width 0) (type default))
   )
+  (wire (pts (xy 48.26 83.82) (xy 48.26 110.49))
+    (stroke (width 0) (type default))
+  )
+  (wire (pts (xy 48.26 53.34) (xy 48.26 78.74))
+    (stroke (width 0) (type default))
+  )
   (wire (pts (xy 254 130.81) (xy 243.84 130.81))
     (stroke (width 0) (type default))
@@
     (stroke (width 0) (type default))
   )
-  (label "AUDIO_IN_L" (at 62.23 53.34 180) (fields_autoplaced)
+  (label "AUDIO_IN_L" (at 68.58 53.34 180) (fields_autoplaced)
     (effects (font (size 1.27 1.27)) (justify right bottom))
   )
-  (label "AUDIO_IN_R" (at 58.42 107.95 180) (fields_autoplaced)
+  (label "AUDIO_IN_R" (at 68.58 107.95 180) (fields_autoplaced)
     (effects (font (size 1.27 1.27)) (justify right bottom))
   )
@@
         (path "/16e2fedd-ee7e-47fb-90b7-873830aa53a9/88ab5ded-31c1-43ab-b0f2-1093ff8b5c31"
           (reference "R29") (unit 1)
+        )
+      )
+    )
+  )
+  (symbol (lib_id "Device:R_Small") (at 53.34 81.28 0) (unit 1)
+    (in_bom yes) (on_board yes) (dnp no) (fields_autoplaced)
+    (property "Reference" "R52" (at 55.88 80.01 0)
+      (effects (font (size 1.27 1.27)) (justify left))
+    )
+    (property "Value" "0R" (at 55.88 82.55 0)
+      (effects (font (size 1.27 1.27)) (justify left))
+    )
+    (property "Footprint" "Resistor_SMD:R_0603_1608Metric" (at 53.34 81.28 0)
+      (effects (font (size 1.27 1.27)) hide)
+    )
+    (property "Datasheet" "~" (at 53.34 81.28 0)
+      (effects (font (size 1.27 1.27)) hide)
+    )
+    (pin "1")
+    (pin "2")
+    (instances
+      (project "Echo Cinematic"
+        (path "/16e2fedd-ee7e-47fb-90b7-873830aa53a9/88ab5ded-31c1-43ab-b0f2-1093ff8b5c31"
+          (reference "R52") (unit 1)
         )
       )
@@
         )
       )
+    )
+  )
+  (symbol (lib_id "Device:R_Small") (at 48.26 81.28 0) (unit 1)
+    (in_bom yes) (on_board yes) (dnp no) (fields_autoplaced)
+    (property "Reference" "R51" (at 45.72 80.01 0)
+      (effects (font (size 1.27 1.27)) (justify right))
+    )
+    (property "Value" "0R" (at 45.72 82.55 0)
+      (effects (font (size 1.27 1.27)) (justify right))
+    )
+    (property "Footprint" "Resistor_SMD:R_0603_1608Metric" (at 48.26 81.28 0)
+      (effects (font (size 1.27 1.27)) hide)
+    )
+    (property "Datasheet" "~" (at 48.26 81.28 0)
+      (effects (font (size 1.27 1.27)) hide)
+    )
+    (pin "1")
+    (pin "2")
+    (instances
+      (project "Echo Cinematic"
+        (path "/16e2fedd-ee7e-47fb-90b7-873830aa53a9/88ab5ded-31c1-43ab-b0f2-1093ff8b5c31"
+          (reference "R51") (unit 1)
+        )
+      )
